Commit message: sim dung JointGroupVelocityController

File: mobile_description/my_mobilerobot/urdf/gazebo_ros2_control.xacro (robot description, xacro)
@@ -1,16 +1,4 @@
 <?xml version="1.0"?>
 <robot xmlns:xacro="http://www.ros.org/wiki/xacro">
-  <!-- =====================================================================
-       ROS2_CONTROL cho robot THẬT (không dùng Gazebo).
-       Plugin my_robot_hardware/MyRobotHardware giao tiếp serial với ESP32.
-       Các tham số dùng xacro arg (khai báo ở my_robot.urdf.xacro) để có thể
-       ghi đè từ dòng lệnh hoặc launch mà không cần sửa file này.
-       [GHI CHÚ 2026-10-13] File này trước đây gộp chung cả phần Gazebo (3 thẻ
-       <gazebo reference=...> đặt ma sát bánh xe + plugin gz_ros2_control-system +
-       hardware gz_ros2_control/GazeboSimSystem). Nay phần của Gazebo đã được
-       CHUYỂN sang file mới gazebo_sim_control.xacro, KHÔNG BỊ XOÁ, chỉ dời đi cho
-       gọn. File này hiện chỉ giữ phần robot thật. Muốn chạy Gazebo thì dùng
-       my_robot.urdf.xacro với use_gazebo true.
-       ===================================================================== -->
   <ros2_control name="MobileBaseHardwareInterface" type="system">
     <!-- <hardware>
@@ -22,14 +10,22 @@
     </hardware> -->
     <hardware>
-      <plugin>mock_components/GenericSystem</plugin>
-      <param name="calculate_dynamics">true</param>
+      <!-- <plugin>mock_components/GenericSystem</plugin>
+      <param name="calculate_dynamics">true</param> -->
+      <plugin>gz_ros2_control/GazeboSimSystem</plugin>
+      <!--gazebosimsystem chay dong co ao thay vi dung dong co that-->
   </hardware>
     <joint name="right_wheel_joint">
-      <command_interface name="velocity" />
+      <command_interface name="velocity">
+       <param name="min">-1</param>
+        <param name="max">1</param>
+      </command_interface>
       <state_interface name="position" />
       <state_interface name="velocity" />
     </joint>
     <joint name="left_wheel_joint">
-      <command_interface name="velocity" />
+      <command_interface name="velocity">
+        <param name="min">-1</param>
+        <param name="max">1</param>
+      </command_interface>
       <state_interface name="position" />
       <state_interface name="velocity" />

File: mobile_description/my_mobilerobot/urdf/gazebo_sim_control.xacro (robot description, xacro)
@@ -1,16 +1,4 @@
 <?xml version="1.0"?>
 <robot xmlns:xacro="http://www.ros.org/wiki/xacro">
-  <!-- =====================================================================
-       ROS2_CONTROL + CẢM BIẾN cho mô phỏng Gazebo (chỉ dùng khi use_gazebo true).
-       [MỚI 2026-10-13] File này được TÁCH RA TỪ gazebo_ros2_control.xacro để giữ
-       nguyên phần dành cho Gazebo (các thẻ <gazebo reference=...> đặt ma sát bánh,
-       plugin gz_ros2_control-system và hardware gz_ros2_control/GazeboSimSystem).
-       Nội dung KHÔNG bị mất, chỉ dời sang file này cho gọn và để file
-       gazebo_ros2_control.xacro lo phần robot thật.
-       Plugin phần cứng gz_ros2_control/GazeboSimSystem (bánh quay trong vật lý Gazebo).
-       Plugin gz_ros2_control-system nạp ros2_control vào Gazebo và trỏ tới
-       mobile_controller/config/controller.yaml.
-       Thẻ gazebo reference dùng để cài ma sát bánh xe giúp robot bám đường.
-       ===================================================================== -->
   <gazebo reference="left_wheel">
     <mu1>1.0</mu1>
@@ -41,27 +29,8 @@
   <gazebo>
     <plugin filename="gz_ros2_control-system" name="gz_ros2_control::GazeboSimROS2ControlPlugin">
-      <parameters>$(find mobile_controller)/config/controller.yaml</parameters>
+<!--plugin cap he thong cua gazebo, cho biet tich hop ros2_control vao moi truong.
+Khi gazebo nap plugin nay se tu dong tao /controller_manager va doc file yaml de bt can quan ly nhung gi-->
+    <parameters>$(find mobile_controller)/config/controller.yaml</parameters>
     </plugin>
   </gazebo>
-  <ros2_control name="RobotSystem" type="system">
-    <hardware>
-      <plugin>gz_ros2_control/GazeboSimSystem</plugin>
-  </hardware>
-    <joint name="right_wheel_joint">
-      <command_interface name="velocity">
-        <param name="min">-1</param>
-        <param name="max">1</param>
-      </command_interface>
-      <state_interface name="position" />
-      <state_interface name="velocity" />
-    </joint>
-    <joint name="left_wheel_joint">
-      <command_interface name="velocity">
-        <param name="min">-1</param>
-        <param name="max">1</param>
-      </command_interface>
-      <state_interface name="position" />
-      <state_interface name="velocity" />
-    </joint>
-  </ros2_control>
 </robot>

File: mobile_description/my_mobilerobot/urdf/my_robot.urdf.xacro (robot description, xacro)
@@ -11,10 +11,6 @@
     <xacro:property name="caster_radius" value="0.05" />
     <xacro:include filename="common_properties.xacro"/>
-    <xacro:if value="$(arg use_gazebo)">
-        <xacro:include filename="gazebo_sim_control.xacro"/>
-    </xacro:if>
-    <xacro:unless value="$(arg use_gazebo)">
-        <xacro:include filename="gazebo_ros2_control.xacro"/>
-    </xacro:unless>
+    <xacro:include filename="gazebo_sim_control.xacro"/>
+    <xacro:include filename="gazebo_ros2_control.xacro"/>
     <xacro:include filename="camera.xacro"/>
     <xacro:include filename="lidar.xacro"/>
